File: Kicad_files/BMS.kicad_sch (KiCad schematic)
At the start: 22 parts, among them J1 USB_B_Mini, Q1 SQJ418EP-T1_GE3, Q2 SQJ418EP-T1_GE3, Q3 SQJ418EP-T1_GE3, U1 BQ297xy, U2 MCP73831-2-OT

Commit message: new kicad files to reflect v1.1 changes
Parts:
- added R7: 10000, Resistor_SMD:R_0805_2012Metric_Pad1.20x1.40mm_HandSolder, symbol Device:R_Small
- Q1, Q2: value SQJ418EP-T1_GE3 -> NMOS
- Q3: value SQJ418EP-T1_GE3 -> PMOS
- renumbered IN+ to IN+1, IN- to IN-1, OUT+ to OUT+1, OUT- to OUT-1
Connections:
- net VP_BATT_NEG is gone; now on net GND: OUT-1.1 (Pin_1), Q1.1 (S_1), Q1.2 (S_2), Q1.3 (S_3), R1.1
- net GND: now also R7.1; no longer C3.2, IN-1.1 (Pin_1), Q2.1 (S_1), Q2.2 (S_2), Q2.3 (S_3), U1.4 (VSS)
- net at Q3.4 (G), R6.2: now also R7.2
- new net V_BAT_NEG: C3.2, IN-1.1 (Pin_1), Q2.1 (S_1), Q2.2 (S_2), Q2.3 (S_3), U1.4 (VSS)
Other:
- note added: "Charging circuit"
- note added: "Protection circuit"
- note added: "USB power"
- moved on the sheet: IN-1, R6
